File: Qi_Rx_STWLC68_throu_hole/Rx.brd (EAGLE design)
At the start: 101.6 x 76.2 mm, 44 parts, among them IC1 STWLC68JRH

Commit message: Rx through-hole cleanup
Parts:
- added TP15, TP16, TP17: TPPAD1-13, testpad:P1-13
- TP14: value PTR1PAD1-13 -> TPPAD1-13
- renumbered TP19 to TP14
Connections:
- new net N$11: R3.2, R4.2, R5.2, TP14.TP
- net GND: now also TP16.TP, TP17.TP
- net V18: now also TP15.TP; no longer R3.2, R4.2, R5.2, TP14.TP
Routing:
- net V18: track 142.3 -> 76.5 mm
- net N$11: track 0.00 -> 21.8 mm
Other:
- board text added: "GND"
- board text added: "INT"
- board text added: "Qi-PRx-STWLC68 2022-11-03"
- board text added: "SCL"
- board text added: "SDA"
- board text added: "V18"
- board text added: "V5"
- board text added: "VI2C"
- board text added: "VOUT"
- board text added: "VRECT"
