File: Qi_Rx_STWLC68_throu_hole/Rx.sch (EAGLE design)
At the start: 44 parts, among them IC1 STWLC68JRH

Commit message: Rx through-hole cleanup
Parts:
- removed TP19: PTR1PAD1-13, testpad:PTR1PAD1-13
- added TP14, TP15, TP16, TP17: TPPAD1-13, testpad:TPPAD1-13
Connections:
- new net N$11: R3.2, R4.2, R5.2, TP14.TP
- net GND: now also TP16.TP, TP17.TP
- net V18: now also TP15.TP; no longer R3.2, R4.2, R5.2, TP19.TP
Other:
- note added: "001"
- note added: "2022WP-Rx-ThrouHole"
- note added: "Design for Qi PRx using STWLC68."
Changed lines of the file:
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@@
 <part name="SUPPLY7" library="supply2" library_urn="urn:adsk.eagle:library:372" deviceset="GND" device=""/>
 <part name="SUPPLY8" library="supply2" library_urn="urn:adsk.eagle:library:372" deviceset="GND" device=""/>
-<part name="TP19" library="testpad" library_urn="urn:adsk.eagle:library:385" deviceset="PTR1" device="PAD1-13" package3d_urn="urn:adsk.eagle:package:27946/1"/>
 <part name="JP1" library="pinhead" library_urn="urn:adsk.eagle:library:325" deviceset="PINHD-1X6" device="" package3d_urn="urn:adsk.eagle:package:22472/2"/>
 <part name="TP1" library="testpad" library_urn="urn:adsk.eagle:library:385" deviceset="TP" device="PAD1-13" package3d_urn="urn:adsk.eagle:package:27946/1"/>
@@
 <part name="U$1" library="SamacSys_Parts" deviceset="SA16A-E3/54" device=""/>
 <part name="U$2" library="SamacSys_Parts" deviceset="SA16A-E3/54" device=""/>
+<part name="FRAME1" library="frames" library_urn="urn:adsk.eagle:library:229" deviceset="LETTER_L" device=""/>
+<part name="TP14" library="testpad" library_urn="urn:adsk.eagle:library:385" deviceset="TP" device="PAD1-13" package3d_urn="urn:adsk.eagle:package:27946/1"/>
+<part name="TP15" library="testpad" library_urn="urn:adsk.eagle:library:385" deviceset="TP" device="PAD1-13" package3d_urn="urn:adsk.eagle:package:27946/1"/>
+<part name="TP16" library="testpad" library_urn="urn:adsk.eagle:library:385" deviceset="TP" device="PAD1-13" package3d_urn="urn:adsk.eagle:package:27946/1"/>
+<part name="TP17" library="testpad" library_urn="urn:adsk.eagle:library:385" deviceset="TP" device="PAD1-13" package3d_urn="urn:adsk.eagle:package:27946/1"/>
 </parts>
 <sheets>
 <sheet>
 <plain>
+<text x="147.066" y="-24.892" size="2.54" layer="94">2022WP-Rx-ThrouHole</text>
+<text x="198.12" y="-25.4" size="2.54" layer="94">001</text>
+<text x="109.22" y="-2.54" size="2.54" layer="94">Design for Qi PRx using STWLC68.</text>
 </plain>
 <instances>
@@
 <attribute name="VALUE" x="122.555" y="4.445" size="1.778" layer="96"/>
 </instance>
-<instance part="TP19" gate="G$1" x="96.52" y="144.78" smashed="yes" rot="R180">
-<attribute name="NAME" x="97.536" y="151.13" size="1.778" layer="95" rot="R270"/>
-<attribute name="TP_SIGNAL_NAME" x="95.25" y="147.32" size="1.778" layer="97" rot="R180"/>
-</instance>
 <instance part="JP1" gate="A" x="-10.16" y="121.92" smashed="yes" rot="MR0">
 <attribute name="NAME" x="-3.81" y="132.715" size="1.778" layer="95" rot="MR0"/>
@@
 </instance>
 <instance part="TP7" gate="G$1" x="58.42" y="127" smashed="yes" rot="R90">
-<attribute name="NAME" x="57.15" y="125.73" size="1.778" layer="95" rot="R90"/>
+<attribute name="NAME" x="57.15" y="125.73" size="1.778" layer="95" rot="R180"/>
 <attribute name="TP_SIGNAL_NAME" x="59.69" y="128.27" size="1.778" layer="97" rot="R90"/>
 </instance>
 <instance part="TP8" gate="G$1" x="58.42" y="129.54" smashed="yes" rot="R90">
-<attribute name="NAME" x="57.15" y="128.27" size="1.778" layer="95" rot="R90"/>
+<attribute name="NAME" x="57.15" y="128.27" size="1.778" layer="95" rot="R180"/>
 <attribute name="TP_SIGNAL_NAME" x="59.69" y="130.81" size="1.778" layer="97" rot="R90"/>
 </instance>
 <instance part="TP9" gate="G$1" x="58.42" y="132.08" smashed="yes" rot="R90">
-<attribute name="NAME" x="57.15" y="130.81" size="1.778" layer="95" rot="R90"/>
+<attribute name="NAME" x="57.15" y="130.81" size="1.778" layer="95" rot="R180"/>
 <attribute name="TP_SIGNAL_NAME" x="59.69" y="133.35" size="1.778" layer="97" rot="R90"/>
 </instance>
 <instance part="TP10" gate="G$1" x="58.42" y="134.62" smashed="yes" rot="R90">
-<attribute name="NAME" x="57.15" y="133.35" size="1.778" layer="95" rot="R90"/>
+<attribute name="NAME" x="57.15" y="133.35" size="1.778" layer="95" rot="R180"/>
 <attribute name="TP_SIGNAL_NAME" x="59.69" y="135.89" size="1.778" layer="97" rot="R90"/>
 </instance>
@@
 <instance part="U$1" gate="G$1" x="-17.78" y="50.8" smashed="yes"/>
 <instance part="U$2" gate="G$1" x="-17.78" y="45.72" smashed="yes"/>
+<instance part="FRAME1" gate="G$1" x="-40.64" y="-33.02" smashed="yes"/>
+<instance part="FRAME1" gate="G$2" x="106.68" y="-33.02" smashed="yes">
+<attribute name="LAST_DATE_TIME" x="119.38" y="-31.75" size="2.54" layer="94"/>
+<attribute name="SHEET" x="193.04" y="-31.75" size="2.54" layer="94"/>
+<attribute name="DRAWING_NAME" x="124.46" y="-13.97" size="2.54" layer="94"/>
+</instance>
+<instance part="TP14" gate="G$1" x="116.84" y="137.16" smashed="yes">
+<attribute name="NAME" x="115.57" y="138.43" size="1.778" layer="95"/>
+<attribute name="TP_SIGNAL_NAME" x="118.11" y="135.89" size="1.778" layer="97"/>
+</instance>
+<instance part="TP15" gate="G$1" x="139.7" y="30.48" smashed="yes" rot="R270">
+<attribute name="NAME" x="140.97" y="31.75" size="1.778" layer="95" rot="R270"/>
+<attribute name="TP_SIGNAL_NAME" x="138.43" y="29.21" size="1.778" layer="97" rot="R270"/>
+</instance>
+<instance part="TP16" gate="G$1" x="78.74" y="127" smashed="yes" rot="R270">
+<attribute name="NAME" x="80.01" y="128.27" size="1.778" layer="95" rot="R270"/>
+<attribute name="TP_SIGNAL_NAME" x="77.47" y="125.73" size="1.778" layer="97" rot="R270"/>
+</instance>
+<instance part="TP17" gate="G$1" x="68.58" y="124.46" smashed="yes" rot="R180">
+<attribute name="NAME" x="69.85" y="123.19" size="1.778" layer="95" rot="R270"/>
+<attribute name="TP_SIGNAL_NAME" x="67.31" y="125.73" size="1.778" layer="97" rot="R180"/>
+</instance>
 </instances>
 <busses>
@@
 </segment>
 <segment>
-<wire x1="60.96" y1="127" x2="76.2" y2="127" width="0.1524" layer="91"/>
+<wire x1="60.96" y1="127" x2="68.58" y2="127" width="0.1524" layer="91"/>
 <label x="66.04" y="127" size="1.778" layer="95"/>
 <pinref part="TP7" gate="G$1" pin="TP"/>
+<pinref part="TP16" gate="G$1" pin="TP"/>
+<pinref part="TP17" gate="G$1" pin="TP"/>
+<wire x1="68.58" y1="127" x2="76.2" y2="127" width="0.1524" layer="91"/>
+<junction x="68.58" y="127"/>
 </segment>
 <segment>
@@
 <net name="V18" class="0">
 <segment>
-<wire x1="93.98" y1="129.54" x2="96.52" y2="129.54" width="0.1524" layer="91"/>
-<wire x1="96.52" y1="129.54" x2="96.52" y2="132.08" width="0.1524" layer="91"/>
-<wire x1="96.52" y1="132.08" x2="96.52" y2="134.62" width="0.1524" layer="91"/>
-<wire x1="96.52" y1="134.62" x2="96.52" y2="142.24" width="0.1524" layer="91"/>
-<wire x1="93.98" y1="134.62" x2="96.52" y2="134.62" width="0.1524" layer="91"/>
-<junction x="96.52" y="134.62"/>
-<wire x1="93.98" y1="132.08" x2="96.52" y2="132.08" width="0.1524" layer="91"/>
-<junction x="96.52" y="132.08"/>
-<label x="96.52" y="142.24" size="1.778" layer="95"/>
-<pinref part="TP19" gate="G$1" pin="TP"/>
-<pinref part="R3" gate="G$1" pin="2"/>
-<pinref part="R4" gate="G$1" pin="2"/>
-<pinref part="R5" gate="G$1" pin="2"/>
-</segment>
-<segment>
 <pinref part="IC1" gate="G$1" pin="RSTB"/>
 <wire x1="88.9" y1="-2.54" x2="93.98" y2="-2.54" width="0.1524" layer="91"/>
@@
 </segment>
 <segment>
-<wire x1="137.16" y1="33.02" x2="137.16" y2="27.94" width="0.1524" layer="91"/>
+<wire x1="137.16" y1="33.02" x2="137.16" y2="30.48" width="0.1524" layer="91"/>
 <label x="134.62" y="30.48" size="1.778" layer="95"/>
 <pinref part="C13" gate="G$1" pin="2"/>
 <pinref part="R6" gate="G$1" pin="1"/>
+<pinref part="TP15" gate="G$1" pin="TP"/>
+<wire x1="137.16" y1="30.48" x2="137.16" y2="27.94" width="0.1524" layer="91"/>
+<junction x="137.16" y="30.48"/>
 </segment>
 <segment>
@@
 </segment>
 </net>
+<net name="N$11" class="0">
+<segment>
+<pinref part="R3" gate="G$1" pin="2"/>
+<pinref part="TP14" gate="G$1" pin="TP"/>
+<wire x1="93.98" y1="134.62" x2="99.06" y2="134.62" width="0.1524" layer="91"/>
+<pinref part="R4" gate="G$1" pin="2"/>
+<wire x1="99.06" y1="134.62" x2="116.84" y2="134.62" width="0.1524" layer="91"/>
+<wire x1="93.98" y1="132.08" x2="99.06" y2="132.08" width="0.1524" layer="91"/>
+<wire x1="99.06" y1="132.08" x2="99.06" y2="134.62" width="0.1524" layer="91"/>
+<junction x="99.06" y="134.62"/>
+<pinref part="R5" gate="G$1" pin="2"/>
+<wire x1="93.98" y1="129.54" x2="99.06" y2="129.54" width="0.1524" layer="91"/>
+<wire x1="99.06" y1="129.54" x2="99.06" y2="132.08" width="0.1524" layer="91"/>
+<junction x="99.06" y="132.08"/>
+</segment>
+</net>
